Commit message: Create dummy launcher with multiple controllers

File: urdf/pointer_car.xacro (robot description, xacro)
@@ -12,4 +12,5 @@
   <xacro:property name="pointer_radius" value="0.05" />
   <xacro:property name="wheel_reduction" value="1" />
+  <xacro:property name="pointer_reduction" value="1" />
   <!-- INCLUDE HELPER SNIPPETS -->
   <xacro:include filename="$(find ros_control_tests)/urdf/snippets.xacro"/>
@@ -55,4 +56,5 @@
     <axis xyz="1 0 0"/>
   </joint>
+  <xacro:transmission_macro joint="pointer_joint" reduction="${pointer_reduction}"/>
   <joint name="pointer_tip_joint" type="fixed">
     <parent link="pointer_link"/>
